File: antic_switch.kicad_pcb (KiCad board)
At the start: 2 copper layers, 47 x 53.3 mm, 11 parts, among them J1 2.54, J2 2.00, P1 ANTIC_Conn, U1 ANTIC_NTSC, U2 74LS245, U3 ANTIC_PAL, U4 74LS245

Commit message: gerber
Parts:
- added J3: 2.54, Connector_PinHeader_2.54mm:PinHeader_2x05_P2.54mm_Horizontal, F.Cu at (142.2, 81.3)
Routing:
- net VCC: track 107.2 -> 112.4 mm
- net /PAL: track 76.1 -> 79.0 mm
- net /NTSC: track 77.0 -> 79.9 mm
- net /~{RESET}: track 71.1 -> 72.7 mm
- net GND: vias 8 -> 12
Other:
- board size 47 x 53.3 mm -> 47.2 x 53.3 mm
- board text added: "Switch"
- board text added: "protoboard"

Commit message: complete rework
Parts:
- J1: value 2.54 -> 2.54m
- J2: value 2.00 -> 2.00m
- moved U2 7.62 mm to (106.7, 55.9)
- moved U4 7.62 mm to (129.5, 55.9)
Connections:
- J1 pad 1: /PAL -> /~{PAL/N_OFF}
- J1 pad 3: /NTSC -> /~{NTSC/P_OFF}
- J2 pad 1: /NTSC -> /~{NTSC/P_OFF}
- J2 pad 3: /PAL -> /~{PAL/N_OFF}
- P1 pad 14: /R/~{W} -> Net-(P1A-R/~{W})
- P1 pad 35: Net-(P1A-FI0) -> /FI0
- P1 pad 4: Net-(P1A-~{LP}) -> /~{LP}
- R1 pad 2: /PAL -> /~{PAL/N_OFF}
- R2 pad 2: /NTSC -> /~{NTSC/P_OFF}
- U1 pad 14: Net-(U1-R/~{W}) -> Net-(P1A-R/~{W})
- U1 pad 35: Net-(P1A-FI0) -> Net-(U1-FI0)
- U1 pad 36: /PAL -> /~{PAL/N_OFF}
- U1 pad 4: Net-(P1A-~{LP}) -> Net-(U1-~{LP})
- U2 pad 11: /PAL -> Net-(U1-~{READY})
- U2 pad 12: Net-(U1-~{READY}) -> /R/~{W}
- U2 pad 13: unconnected-(U2-B5-Pad13) -> Net-(U1-~{HALT})
- U2 pad 14: unconnected-(U2-B4-Pad14) -> Net-(U1-~{REF})
- U2 pad 15: /R/~{W} -> Net-(U1-~{NMI})
- U2 pad 16: Net-(U1-~{HALT}) -> /FI0
- U2 pad 17: Net-(U1-~{REF}) -> /~{RESET}
- U2 pad 18: Net-(U1-~{NMI}) -> /~{LP}
- U2 pad 19: /NTSC -> /~{NTSC/P_OFF}
- U2 pad 2: /~{NMI} -> Net-(U1-~{LP})
- U2 pad 3: /~{REF} -> /~{NTSC/P_OFF}
- U2 pad 4: /~{HALT} -> Net-(U1-FI0)
- U2 pad 5: Net-(U1-R/~{W}) -> /~{NMI}
- U2 pad 6: unconnected-(U2-A4-Pad6) -> /~{REF}
- U2 pad 7: unconnected-(U2-A5-Pad7) -> /~{HALT}
- U2 pad 8: /~{READY} -> unconnected-(U2-A6-Pad8)
- U2 pad 9: /~{RESET} -> /~{READY}
- U3 pad 14: Net-(U3B-R/~{W}) -> Net-(P1A-R/~{W})
- U3 pad 35: Net-(P1A-FI0) -> Net-(U3B-FI0)
- U3 pad 36: /NTSC -> /~{NTSC/P_OFF}
- U3 pad 4: Net-(P1A-~{LP}) -> Net-(U3B-~{LP})
- U4 pad 11: /NTSC -> Net-(U3B-~{READY})
- U4 pad 12: Net-(U3B-~{READY}) -> /R/~{W}
- U4 pad 13: unconnected-(U4-B5-Pad13) -> Net-(U3B-~{HALT})
- U4 pad 14: unconnected-(U4-B4-Pad14) -> Net-(U3B-~{REF})
- U4 pad 15: /R/~{W} -> Net-(U3B-~{NMI})
- U4 pad 16: Net-(U3B-~{HALT}) -> /FI0
- U4 pad 17: Net-(U3B-~{REF}) -> /~{RESET}
- U4 pad 18: Net-(U3B-~{NMI}) -> /~{LP}
- U4 pad 19: /PAL -> /~{PAL/N_OFF}
- U4 pad 2: /~{NMI} -> Net-(U3B-~{LP})
- U4 pad 3: /~{REF} -> /~{PAL/N_OFF}
- U4 pad 4: /~{HALT} -> Net-(U3B-FI0)
- U4 pad 5: Net-(U3B-R/~{W}) -> /~{NMI}
- U4 pad 6: unconnected-(U4-A4-Pad6) -> /~{REF}
- U4 pad 7: unconnected-(U4-A5-Pad7) -> /~{HALT}
- U4 pad 8: /~{READY} -> unconnected-(U4-A6-Pad8)
- U4 pad 9: /~{RESET} -> /~{READY}
Routing:
- net /NTSC: track 79.9 -> 0.00 mm, vias 1 -> 0
- net /PAL: track 79.0 -> 0.00 mm, vias 1 -> 0
- net /~{PAL/N_OFF}: track 0.00 -> 75.2 mm, vias 0 -> 2
- net /~{NTSC/P_OFF}: track 0.00 -> 73.0 mm
- net /~{LP}: track 0.00 -> 57.0 mm, vias 0 -> 3
- net /~{REF}: track 29.9 -> 83.3 mm, vias 0 -> 3
- net /~{RESET}: track 72.7 -> 28.4 mm, vias 0 -> 1
- net Net-(P1A-R/~{W}): track 0.00 -> 37.3 mm
- net Net-(P1A-D7): track 23.8 -> 56.1 mm, vias 0 -> 1
- net Net-(P1A-FI0): track 30.3 -> 0.00 mm, vias 1 -> 0
- net /FI0: track 0.00 -> 25.6 mm
- net GND: track 34.2 -> 8.67 mm, vias 12 -> 9
- net Net-(P1A-~{LP}): track 23.8 -> 0.00 mm
- net unconnected-(U4-A6-Pad8): track 0.00 -> 23.7 mm
- net /R/~{W}: track 51.8 -> 31.3 mm, vias 2 -> 3
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